File: hardware/1335/A1335v1.kicad_pcb (KiCad board)
At the start: 2 copper layers, 50.8 x 50.8 mm, 23 parts, among them J1 TERMINALES1, J2 TERMINALES2

Commit message: add a1335_rev2 files
Parts:
- removed T-MISO1, T-SDA1, T-VCC1: TestPoint, TestPoint:TestPoint_THTPad_2.0x2.0mm_Drill1.0mm
- moved J1 40.7 mm to (195.6, 96.5), turned to 270 degrees
- moved J2 40.6 mm to (236.2, 95.2), turned to 90 degrees
