File: hardware/1335_rev1/1335_rev1.kicad_pcb (KiCad board)
At the start: 2 copper layers, 45 x 45 mm, 21 parts, among them J1 Screw_Terminal_01x05, J2 Screw_Terminal_01x06, U1 A1335

Commit message: Error in boom
Parts:
- C1, C2: footprint Capacitor_Tantalum_SMD:CP_EIA-1608-08_AVX-J -> Capacitor_Tantalum_SMD:CP_EIA-2012-15_AVX-P_Pad1.30x1.05mm_HandSolder
- moved C2 1.27 mm to (137.2, 69.2)
Routing:
- net /BYP: track 36.1 -> 39.7 mm
- net GND: track 23.6 -> 22.4 mm
