File: hardware/1335_rev1/1335_rev1.sch (KiCad schematic (older format))
At the start: 20 parts, among them J1 Screw_Terminal_01x05, J2 Screw_Terminal_01x06, U1 A1335

Commit message: Updates
Other:
- moved on the sheet: C1, H1, H2, H3, H4, U1
Changed lines of the file:
@@
 L Mechanical:MountingHole H1
 U 1 1 6046695B
-P 850 1125
-F 0 "H1" H 950 1171 50  0000 L CNN
-F 1 "MountingHole" H 950 1080 50  0000 L CNN
-F 2 "MountingHole:MountingHole_3.2mm_M3_Pad_Via" H 850 1125 50  0001 C CNN
-F 3 "~" H 850 1125 50  0001 C CNN
-	1    850  1125
+P 900 1050
+F 0 "H1" H 1000 1096 50  0000 L CNN
+F 1 "MountingHole" H 1000 1005 50  0000 L CNN
+F 2 "MountingHole:MountingHole_3.2mm_M3_Pad_Via" H 900 1050 50  0001 C CNN
+F 3 "~" H 900 1050 50  0001 C CNN
+	1    900  1050
 	1    0    0    -1
 $EndComp
@@
 L Mechanical:MountingHole H2
 U 1 1 6046714D
-P 850 1350
-F 0 "H2" H 950 1396 50  0000 L CNN
-F 1 "MountingHole" H 950 1305 50  0000 L CNN
-F 2 "MountingHole:MountingHole_3.2mm_M3_Pad_Via" H 850 1350 50  0001 C CNN
-F 3 "~" H 850 1350 50  0001 C CNN
-	1    850  1350
+P 900 1275
+F 0 "H2" H 1000 1321 50  0000 L CNN
+F 1 "MountingHole" H 1000 1230 50  0000 L CNN
+F 2 "MountingHole:MountingHole_3.2mm_M3_Pad_Via" H 900 1275 50  0001 C CNN
+F 3 "~" H 900 1275 50  0001 C CNN
+	1    900  1275
 	1    0    0    -1
 $EndComp
@@
 L Mechanical:MountingHole H3
 U 1 1 60467542
-P 850 1575
-F 0 "H3" H 950 1621 50  0000 L CNN
-F 1 "MountingHole" H 950 1530 50  0000 L CNN
-F 2 "MountingHole:MountingHole_3.2mm_M3_Pad_Via" H 850 1575 50  0001 C CNN
-F 3 "~" H 850 1575 50  0001 C CNN
-	1    850  1575
+P 900 1500
+F 0 "H3" H 1000 1546 50  0000 L CNN
+F 1 "MountingHole" H 1000 1455 50  0000 L CNN
+F 2 "MountingHole:MountingHole_3.2mm_M3_Pad_Via" H 900 1500 50  0001 C CNN
+F 3 "~" H 900 1500 50  0001 C CNN
+	1    900  1500
 	1    0    0    -1
 $EndComp
@@
 L Mechanical:MountingHole H4
 U 1 1 604678DB
-P 850 1800
-F 0 "H4" H 950 1846 50  0000 L CNN
-F 1 "MountingHole" H 950 1755 50  0000 L CNN
-F 2 "MountingHole:MountingHole_3.2mm_M3_Pad_Via" H 850 1800 50  0001 C CNN
-F 3 "~" H 850 1800 50  0001 C CNN
-	1    850  1800
+P 900 1725
+F 0 "H4" H 1000 1771 50  0000 L CNN
+F 1 "MountingHole" H 1000 1680 50  0000 L CNN
+F 2 "MountingHole:MountingHole_3.2mm_M3_Pad_Via" H 900 1725 50  0001 C CNN
+F 3 "~" H 900 1725 50  0001 C CNN
+	1    900  1725
 	1    0    0    -1
 $EndComp
@@
 L HALL:A1335 U1
 U 1 1 60468B21
-P 2475 2500
-F 0 "U1" H 3125 2765 50  0000 C CNN
-F 1 "A1335" H 3125 2674 50  0000 C CNN
-F 2 "Tssop_14:TSSOP14" H 2366 2650 50  0001 C CNN
-F 3 "" H 2366 2650 50  0001 C CNN
-	1    2475 2500
+P 2750 2550
+F 0 "U1" H 3400 2815 50  0000 C CNN
+F 1 "A1335" H 3400 2724 50  0000 C CNN
+F 2 "Tssop_14:TSSOP14" H 2641 2700 50  0001 C CNN
+F 3 "" H 2641 2700 50  0001 C CNN
+	1    2750 2550
 	1    0    0    -1
 $EndComp
@@
 Text GLabel 3950 1300 0    50   Input ~ 0
 CS
-NoConn ~ 2675 2800
-NoConn ~ 2675 3000
+NoConn ~ 2950 2850
+NoConn ~ 2950 3050
 $Comp
 L power:GND #PWR0105
 U 1 1 60476818
-P 3575 2500
-F 0 "#PWR0105" H 3575 2250 50  0001 C CNN
-F 1 "GND" V 3580 2372 50  0000 R CNN
-F 2 "" H 3575 2500 50  0001 C CNN
-F 3 "" H 3575 2500 50  0001 C CNN
-	1    3575 2500
+P 3850 2550
+F 0 "#PWR0105" H 3850 2300 50  0001 C CNN
+F 1 "GND" V 3855 2422 50  0000 R CNN
+F 2 "" H 3850 2550 50  0001 C CNN
+F 3 "" H 3850 2550 50  0001 C CNN
+	1    3850 2550
 	0    -1   -1   0
 $EndComp
@@
 L power:GND #PWR0106
 U 1 1 60477352
-P 2675 3100
-F 0 "#PWR0106" H 2675 2850 50  0001 C CNN
-F 1 "GND" H 2680 2927 50  0000 C CNN
-F 2 "" H 2675 3100 50  0001 C CNN
-F 3 "" H 2675 3100 50  0001 C CNN
-	1    2675 3100
+P 2950 3150
+F 0 "#PWR0106" H 2950 2900 50  0001 C CNN
+F 1 "GND" H 2955 2977 50  0000 C CNN
+F 2 "" H 2950 3150 50  0001 C CNN
+F 3 "" H 2950 3150 50  0001 C CNN
+	1    2950 3150
 	1    0    0    -1
 $EndComp
@@
 L power:+5V #PWR0107
 U 1 1 60479752
-P 2675 2900
-F 0 "#PWR0107" H 2675 2750 50  0001 C CNN
-F 1 "+5V" V 2690 3028 50  0000 L CNN
-F 2 "" H 2675 2900 50  0001 C CNN
-F 3 "" H 2675 2900 50  0001 C CNN
-	1    2675 2900
+P 2950 2950
+F 0 "#PWR0107" H 2950 2800 50  0001 C CNN
+F 1 "+5V" V 2965 3078 50  0000 L CNN
+F 2 "" H 2950 2950 50  0001 C CNN
+F 3 "" H 2950 2950 50  0001 C CNN
+	1    2950 2950
 	0    -1   -1   0
 $EndComp
@@
 L power:GND #PWR0108
 U 1 1 6047B24B
-P 2675 2700
-F 0 "#PWR0108" H 2675 2450 50  0001 C CNN
-F 1 "GND" V 2680 2572 50  0000 R CNN
-F 2 "" H 2675 2700 50  0001 C CNN
-F 3 "" H 2675 2700 50  0001 C CNN
-	1    2675 2700
+P 2950 2750
+F 0 "#PWR0108" H 2950 2500 50  0001 C CNN
+F 1 "GND" V 2955 2622 50  0000 R CNN
+F 2 "" H 2950 2750 50  0001 C CNN
+F 3 "" H 2950 2750 50  0001 C CNN
+	1    2950 2750
 	0    1    1    0
 $EndComp
@@
 	2350 500  2350 2000
 Wire Wire Line
-	3575 3100 3800 3100
-Text Label 3800 3100 0    59   ~ 0
+	3850 3150 4075 3150
+Text Label 4075 3150 0    59   ~ 0
 ISEL
 Text Label 6025 1600 0    59   ~ 0
 ISEL
 Wire Wire Line
-	3575 2600 3775 2600
-Wire Wire Line
-	3775 2700 3575 2700
-Wire Wire Line
-	3575 2800 3775 2800
-Wire Wire Line
-	3575 2900 3775 2900
-Text Label 1975 2600 0    59   ~ 0
+	3850 2650 4050 2650
+Wire Wire Line
+	4050 2750 3850 2750
+Wire Wire Line
+	3850 2850 4050 2850
+Wire Wire Line
+	3850 2950 4050 2950
+Text Label 2250 2650 0    59   ~ 0
 BYP
-Text Label 3775 2600 0    59   ~ 0
+Text Label 4050 2650 0    59   ~ 0
 SA0-CS
-Text Label 3775 2700 0    59   ~ 0
+Text Label 4050 2750 0    59   ~ 0
 SA1-MOSI
-Text Label 3775 2800 0    59   ~ 0
+Text Label 4050 2850 0    59   ~ 0
 SCL-CLK
-Text Label 3775 2900 0    59   ~ 0
+Text Label 4050 2950 0    59   ~ 0
 SDA-MISO
 $Comp
 L power:GND #PWR0110
 U 1 1 604837F9
-P 2475 2500
-F 0 "#PWR0110" H 2475 2250 50  0001 C CNN
-F 1 "GND" V 2480 2372 50  0000 R CNN
-F 2 "" H 2475 2500 50  0001 C CNN
-F 3 "" H 2475 2500 50  0001 C CNN
-	1    2475 2500
+P 2750 2550
+F 0 "#PWR0110" H 2750 2300 50  0001 C CNN
+F 1 "GND" V 2755 2422 50  0000 R CNN
+F 2 "" H 2750 2550 50  0001 C CNN
+F 3 "" H 2750 2550 50  0001 C CNN
+	1    2750 2550
 	0    1    1    0
 $EndComp
@@
 L power:GND #PWR0111
 U 1 1 604847D8
-P 1975 2925
-F 0 "#PWR0111" H 1975 2675 50  0001 C CNN
-F 1 "GND" H 1980 2752 50  0000 C CNN
-F 2 "" H 1975 2925 50  0001 C CNN
-F 3 "" H 1975 2925 50  0001 C CNN
-	1    1975 2925
-	1    0    0    -1
-$EndComp
-Wire Wire Line
-	1975 2600 1975 2625
-Wire Wire Line
-	1975 2600 2675 2600
-Wire Wire Line
-	2475 2500 2675 2500
+P 2250 2975
+F 0 "#PWR0111" H 2250 2725 50  0001 C CNN
+F 1 "GND" H 2255 2802 50  0000 C CNN
+F 2 "" H 2250 2975 50  0001 C CNN
+F 3 "" H 2250 2975 50  0001 C CNN
+	1    2250 2975
+	1    0    0    -1
+$EndComp
+Wire Wire Line
+	2250 2650 2250 2675
+Wire Wire Line
+	2250 2650 2950 2650
+Wire Wire Line
+	2750 2550 2950 2550
 Text Label 5550 1400 2    59   ~ 0
 BYP
@@
 L Device:CP1 C1
 U 1 1 6049E44B
-P 1975 2775
-F 0 "C1" H 2090 2821 50  0000 L CNN
-F 1 "100n" H 2090 2730 50  0000 L CNN
-F 2 "Capacitor_Tantalum_SMD:CP_EIA-1608-08_AVX-J" H 1975 2775 50  0001 C CNN
-F 3 "~" H 1975 2775 50  0001 C CNN
-	1    1975 2775
+P 2250 2825
+F 0 "C1" H 2365 2871 50  0000 L CNN
+F 1 "100n" H 2365 2780 50  0000 L CNN
+F 2 "Capacitor_Tantalum_SMD:CP_EIA-1608-08_AVX-J" H 2250 2825 50  0001 C CNN
+F 3 "~" H 2250 2825 50  0001 C CNN
+	1    2250 2825
 	1    0    0    -1
 $EndComp
@@
 	-1   0    0    1
 $EndComp
-NoConn ~ 3575 3000
+NoConn ~ 3850 3050
 Wire Notes Line
 	5000 4900 525  4900

Commit message: Updates in pcb
Other:
- note added: "Power LED indicator"
- note added: "Pull up resistor for I2C"
- moved on the sheet: D1, R1, R2, R3
Changed lines of the file:
@@
 encoding utf-8
 Sheet 1 1
-Title ""
-Date ""
-Rev ""
-Comp ""
-Comment1 ""
-Comment2 ""
-Comment3 ""
-Comment4 ""
+Title "A1335 Allegro Sensor Board"
+Date "2021-03-29"
+Rev "2.0"
+Comp "FIUNER - LIRINS"
+Comment1 "Se implementaron los protocolos SPI e I2C. Falta incorporar el protocolo SENT."
+Comment2 "Se mejoro la organizacón del esquematico de la v1.1"
+Comment3 "Los pines estan agrupados de acuerdo al protocolo de comunicación"
+Comment4 "Se añaden los Mounting Holes"
 $EndDescr
 Text Notes 800  800  0    79   ~ 0
@@
 	1    0    0    -1
 $EndComp
-Text Notes 550  2225 0    59   ~ 0
+Text Notes 650  2400 0    59   ~ 0
 Decoupling capacitor\n
 $Comp
@@
 L power:+5V #PWR0116
 U 1 1 6047ABD4
-P 3825 3650
-F 0 "#PWR0116" H 3825 3500 50  0001 C CNN
-F 1 "+5V" H 3840 3778 50  0000 L CNN
-F 2 "" H 3825 3650 50  0001 C CNN
-F 3 "" H 3825 3650 50  0001 C CNN
-	1    3825 3650
+P 2975 3625
+F 0 "#PWR0116" H 2975 3475 50  0001 C CNN
+F 1 "+5V" H 2990 3753 50  0000 L CNN
+F 2 "" H 2975 3625 50  0001 C CNN
+F 3 "" H 2975 3625 50  0001 C CNN
+	1    2975 3625
 	1    0    0    -1
 $EndComp
@@
 L power:GND #PWR0117
 U 1 1 6047B169
-P 3825 4425
-F 0 "#PWR0117" H 3825 4175 50  0001 C CNN
-F 1 "GND" H 3830 4297 50  0000 R CNN
-F 2 "" H 3825 4425 50  0001 C CNN
-F 3 "" H 3825 4425 50  0001 C CNN
-	1    3825 4425
+P 2975 4400
+F 0 "#PWR0117" H 2975 4150 50  0001 C CNN
+F 1 "GND" H 2980 4272 50  0000 R CNN
+F 2 "" H 2975 4400 50  0001 C CNN
+F 3 "" H 2975 4400 50  0001 C CNN
+	1    2975 4400
 	1    0    0    -1
 $EndComp
@@
 L Device:LED D1
 U 1 1 6047BFDB
-P 3825 4200
-F 0 "D1" V 3864 4082 50  0000 R CNN
-F 1 "LED" V 3773 4082 50  0000 R CNN
-F 2 "LED_SMD:LED_0603_1608Metric" H 3825 4200 50  0001 C CNN
-F 3 "~" H 3825 4200 50  0001 C CNN
-	1    3825 4200
+P 2975 4175
+F 0 "D1" V 3014 4057 50  0000 R CNN
+F 1 "LED" V 2923 4057 50  0000 R CNN
+F 2 "LED_SMD:LED_0603_1608Metric" H 2975 4175 50  0001 C CNN
+F 3 "~" H 2975 4175 50  0001 C CNN
+	1    2975 4175
 	0    -1   -1   0
 $EndComp
@@
 L Device:R R1
 U 1 1 6047CC80
-P 3825 3850
-F 0 "R1" H 3895 3896 50  0000 L CNN
-F 1 "1k" H 3895 3805 50  0000 L CNN
-F 2 "Resistor_SMD:R_0603_1608Metric" V 3755 3850 50  0001 C CNN
-F 3 "~" H 3825 3850 50  0001 C CNN
-	1    3825 3850
-	1    0    0    -1
-$EndComp
-Wire Wire Line
-	3825 3700 3825 3650
-Wire Wire Line
-	3825 4000 3825 4050
-Wire Wire Line
-	3825 4425 3825 4350
+P 2975 3825
+F 0 "R1" H 3045 3871 50  0000 L CNN
+F 1 "1k" H 3045 3780 50  0000 L CNN
+F 2 "Resistor_SMD:R_0603_1608Metric" V 2905 3825 50  0001 C CNN
+F 3 "~" H 2975 3825 50  0001 C CNN
+	1    2975 3825
+	1    0    0    -1
+$EndComp
+Wire Wire Line
+	2975 3675 2975 3625
+Wire Wire Line
+	2975 3975 2975 4025
+Wire Wire Line
+	2975 4400 2975 4325
 $Comp
 L Device:R R3
 U 1 1 604B0FB7
-P 2525 4000
-F 0 "R3" H 2595 4046 50  0000 L CNN
-F 1 "1k" H 2595 3955 50  0000 L CNN
-F 2 "Resistor_SMD:R_0603_1608Metric" V 2455 4000 50  0001 C CNN
-F 3 "~" H 2525 4000 50  0001 C CNN
-	1    2525 4000
+P 1200 4075
+F 0 "R3" H 1270 4121 50  0000 L CNN
+F 1 "1k" H 1270 4030 50  0000 L CNN
+F 2 "Resistor_SMD:R_0603_1608Metric" V 1130 4075 50  0001 C CNN
+F 3 "~" H 1200 4075 50  0001 C CNN
+	1    1200 4075
 	1    0    0    -1
 $EndComp
@@
 L Device:R R2
 U 1 1 604B1BBC
-P 2250 4000
-F 0 "R2" H 2320 4046 50  0000 L CNN
-F 1 "1k" H 2320 3955 50  0000 L CNN
-F 2 "Resistor_SMD:R_0603_1608Metric" V 2180 4000 50  0001 C CNN
-F 3 "~" H 2250 4000 50  0001 C CNN
-	1    2250 4000
+P 925 4075
+F 0 "R2" H 995 4121 50  0000 L CNN
+F 1 "1k" H 995 4030 50  0000 L CNN
+F 2 "Resistor_SMD:R_0603_1608Metric" V 855 4075 50  0001 C CNN
+F 3 "~" H 925 4075 50  0001 C CNN
+	1    925  4075
 	1    0    0    -1
 $EndComp
@@
 	3950 1300 4425 1300
 Wire Wire Line
-	2250 4150 2250 4250
-Wire Wire Line
-	2525 4150 2525 4250
-Wire Wire Line
-	2250 3850 2250 3750
-Wire Wire Line
-	2250 3750 2400 3750
-Wire Wire Line
-	2525 3750 2525 3850
-Connection ~ 2400 3750
-Wire Wire Line
-	2400 3750 2525 3750
+	925  4225 925  4325
+Wire Wire Line
+	1200 4225 1200 4325
+Wire Wire Line
+	925  3925 925  3825
+Wire Wire Line
+	925  3825 1075 3825
+Wire Wire Line
+	1200 3825 1200 3925
+Connection ~ 1075 3825
+Wire Wire Line
+	1075 3825 1200 3825
 $Comp
 L power:+3V3 #PWR0118
 U 1 1 604BB954
-P 2400 3650
-F 0 "#PWR0118" H 2400 3500 50  0001 C CNN
-F 1 "+3V3" H 2415 3778 50  0000 L CNN
-F 2 "" H 2400 3650 50  0001 C CNN
-F 3 "" H 2400 3650 50  0001 C CNN
-	1    2400 3650
+P 1075 3725
+F 0 "#PWR0118" H 1075 3575 50  0001 C CNN
+F 1 "+3V3" H 1090 3853 50  0000 L CNN
+F 2 "" H 1075 3725 50  0001 C CNN
+F 3 "" H 1075 3725 50  0001 C CNN
+	1    1075 3725
 	1    0    0    -1
 $EndComp
@@
 Text Notes 3825 975  0    79   ~ 0
 SPI connectors
-Text GLabel 2300 4250 2    50   Input ~ 0
+Text GLabel 975  4325 2    50   Input ~ 0
 SDA
-Text GLabel 2575 4250 2    50   Input ~ 0
+Text GLabel 1250 4325 2    50   Input ~ 0
 SCL
 Wire Wire Line
-	2575 4250 2525 4250
-Wire Wire Line
-	2300 4250 2250 4250
-Wire Wire Line
-	2400 3750 2400 3650
+	1250 4325 1200 4325
+Wire Wire Line
+	975  4325 925  4325
+Wire Wire Line
+	1075 3825 1075 3725
 $Comp
 L Connector:Screw_Terminal_01x05 J1
@@
 Text Notes 6675 1825 0    59   ~ 0
 1-2\n2-3
+Text Notes 600  3500 0    79   ~ 0
+Pull up resistor for I2C
+Text Notes 3325 3750 0    59   ~ 0
+Power LED indicator
 $EndSCHEMATC

Commit message: Send to review
Esteban Osella aprueba el diseño del PCB
Other:
- moved on the sheet: D1, R1, R2, R3
Changed lines of the file:
@@
 $Descr A4 11693 8268
 encoding utf-8
-Sheet 1 1
+Sheet 1 2
 Title "A1335 Allegro Sensor Board"
 Date "2021-03-29"
@@
 L power:+5V #PWR0116
 U 1 1 6047ABD4
-P 2975 3625
-F 0 "#PWR0116" H 2975 3475 50  0001 C CNN
-F 1 "+5V" H 2990 3753 50  0000 L CNN
-F 2 "" H 2975 3625 50  0001 C CNN
-F 3 "" H 2975 3625 50  0001 C CNN
-	1    2975 3625
+P 3350 3775
+F 0 "#PWR0116" H 3350 3625 50  0001 C CNN
+F 1 "+5V" H 3365 3903 50  0000 L CNN
+F 2 "" H 3350 3775 50  0001 C CNN
+F 3 "" H 3350 3775 50  0001 C CNN
+	1    3350 3775
 	1    0    0    -1
 $EndComp
@@
 L power:GND #PWR0117
 U 1 1 6047B169
-P 2975 4400
-F 0 "#PWR0117" H 2975 4150 50  0001 C CNN
-F 1 "GND" H 2980 4272 50  0000 R CNN
-F 2 "" H 2975 4400 50  0001 C CNN
-F 3 "" H 2975 4400 50  0001 C CNN
-	1    2975 4400
+P 3350 4550
+F 0 "#PWR0117" H 3350 4300 50  0001 C CNN
+F 1 "GND" H 3355 4422 50  0000 R CNN
+F 2 "" H 3350 4550 50  0001 C CNN
+F 3 "" H 3350 4550 50  0001 C CNN
+	1    3350 4550
 	1    0    0    -1
 $EndComp
@@
 L Device:LED D1
 U 1 1 6047BFDB
-P 2975 4175
-F 0 "D1" V 3014 4057 50  0000 R CNN
-F 1 "LED" V 2923 4057 50  0000 R CNN
-F 2 "LED_SMD:LED_0603_1608Metric" H 2975 4175 50  0001 C CNN
-F 3 "~" H 2975 4175 50  0001 C CNN
-	1    2975 4175
+P 3350 4325
+F 0 "D1" V 3389 4207 50  0000 R CNN
+F 1 "LED" V 3298 4207 50  0000 R CNN
+F 2 "LED_SMD:LED_0603_1608Metric" H 3350 4325 50  0001 C CNN
+F 3 "~" H 3350 4325 50  0001 C CNN
+	1    3350 4325
 	0    -1   -1   0
 $EndComp
@@
 L Device:R R1
 U 1 1 6047CC80
-P 2975 3825
-F 0 "R1" H 3045 3871 50  0000 L CNN
-F 1 "1k" H 3045 3780 50  0000 L CNN
-F 2 "Resistor_SMD:R_0603_1608Metric" V 2905 3825 50  0001 C CNN
-F 3 "~" H 2975 3825 50  0001 C CNN
-	1    2975 3825
-	1    0    0    -1
-$EndComp
-Wire Wire Line
-	2975 3675 2975 3625
-Wire Wire Line
-	2975 3975 2975 4025
-Wire Wire Line
-	2975 4400 2975 4325
+P 3350 3975
+F 0 "R1" H 3420 4021 50  0000 L CNN
+F 1 "1k" H 3420 3930 50  0000 L CNN
+F 2 "Resistor_SMD:R_0603_1608Metric" V 3280 3975 50  0001 C CNN
+F 3 "~" H 3350 3975 50  0001 C CNN
+	1    3350 3975
+	1    0    0    -1
+$EndComp
+Wire Wire Line
+	3350 3825 3350 3775
+Wire Wire Line
+	3350 4125 3350 4175
+Wire Wire Line
+	3350 4550 3350 4475
 $Comp
 L Device:R R3
 U 1 1 604B0FB7
-P 1200 4075
-F 0 "R3" H 1270 4121 50  0000 L CNN
-F 1 "1k" H 1270 4030 50  0000 L CNN
-F 2 "Resistor_SMD:R_0603_1608Metric" V 1130 4075 50  0001 C CNN
-F 3 "~" H 1200 4075 50  0001 C CNN
-	1    1200 4075
+P 1375 4175
+F 0 "R3" H 1445 4221 50  0000 L CNN
+F 1 "1k" H 1445 4130 50  0000 L CNN
+F 2 "Resistor_SMD:R_0603_1608Metric" V 1305 4175 50  0001 C CNN
+F 3 "~" H 1375 4175 50  0001 C CNN
+	1    1375 4175
 	1    0    0    -1
 $EndComp
@@
 L Device:R R2
 U 1 1 604B1BBC
-P 925 4075
-F 0 "R2" H 995 4121 50  0000 L CNN
-F 1 "1k" H 995 4030 50  0000 L CNN
-F 2 "Resistor_SMD:R_0603_1608Metric" V 855 4075 50  0001 C CNN
-F 3 "~" H 925 4075 50  0001 C CNN
-	1    925  4075
+P 1100 4175
+F 0 "R2" H 1170 4221 50  0000 L CNN
+F 1 "1k" H 1170 4130 50  0000 L CNN
+F 2 "Resistor_SMD:R_0603_1608Metric" V 1030 4175 50  0001 C CNN
+F 3 "~" H 1100 4175 50  0001 C CNN
+	1    1100 4175
 	1    0    0    -1
 $EndComp
@@
 	3950 1300 4425 1300
 Wire Wire Line
-	925  4225 925  4325
-Wire Wire Line
-	1200 4225 1200 4325
-Wire Wire Line
-	925  3925 925  3825
-Wire Wire Line
-	925  3825 1075 3825
-Wire Wire Line
-	1200 3825 1200 3925
-Connection ~ 1075 3825
-Wire Wire Line
-	1075 3825 1200 3825
+	1100 4325 1100 4425
+Wire Wire Line
+	1375 4325 1375 4425
+Wire Wire Line
+	1100 4025 1100 3925
+Wire Wire Line
+	1100 3925 1250 3925
+Wire Wire Line
+	1375 3925 1375 4025
+Connection ~ 1250 3925
+Wire Wire Line
+	1250 3925 1375 3925
 $Comp
 L power:+3V3 #PWR0118
 U 1 1 604BB954
-P 1075 3725
-F 0 "#PWR0118" H 1075 3575 50  0001 C CNN
-F 1 "+3V3" H 1090 3853 50  0000 L CNN
-F 2 "" H 1075 3725 50  0001 C CNN
-F 3 "" H 1075 3725 50  0001 C CNN
-	1    1075 3725
+P 1250 3825
+F 0 "#PWR0118" H 1250 3675 50  0001 C CNN
+F 1 "+3V3" H 1265 3953 50  0000 L CNN
+F 2 "" H 1250 3825 50  0001 C CNN
+F 3 "" H 1250 3825 50  0001 C CNN
+	1    1250 3825
 	1    0    0    -1
 $EndComp
@@
 Text Notes 3825 975  0    79   ~ 0
 SPI connectors
-Text GLabel 975  4325 2    50   Input ~ 0
+Text GLabel 1150 4425 2    50   Input ~ 0
 SDA
-Text GLabel 1250 4325 2    50   Input ~ 0
+Text GLabel 1425 4425 2    50   Input ~ 0
 SCL
 Wire Wire Line
-	1250 4325 1200 4325
-Wire Wire Line
-	975  4325 925  4325
-Wire Wire Line
-	1075 3825 1075 3725
+	1425 4425 1375 4425
+Wire Wire Line
+	1150 4425 1100 4425
+Wire Wire Line
+	1250 3925 1250 3825
 $Comp
 L Connector:Screw_Terminal_01x05 J1
@@
 NoConn ~ 3850 3050
 Wire Notes Line
-	5000 4900 525  4900
-Wire Notes Line
 	525  4900 525  4875
 Wire Notes Line
@@
 Text Notes 6675 1825 0    59   ~ 0
 1-2\n2-3
-Text Notes 600  3500 0    79   ~ 0
+Text Notes 775  3600 0    79   ~ 0
 Pull up resistor for I2C
-Text Notes 3325 3750 0    59   ~ 0
+Text Notes 2875 3550 0    59   ~ 0
 Power LED indicator
+Wire Notes Line
+	9075 4900 9075 2025
+Wire Notes Line
+	525  4900 9075 4900
+Wire Notes Line
+	9075 2000 9075 475
 $EndSCHEMATC

Commit message: Error in boom
Parts:
- C1, C2: footprint Capacitor_Tantalum_SMD:CP_EIA-1608-08_AVX-J -> Capacitor_Tantalum_SMD:CP_EIA-2012-15_AVX-P_Pad1.30x1.05mm_HandSolder
Changed lines of the file:
@@
 $Descr A4 11693 8268
 encoding utf-8
-Sheet 1 2
+Sheet 1 1
 Title "A1335 Allegro Sensor Board"
 Date "2021-03-29"
@@
 F 0 "C1" H 2365 2871 50  0000 L CNN
 F 1 "100n" H 2365 2780 50  0000 L CNN
-F 2 "Capacitor_Tantalum_SMD:CP_EIA-1608-08_AVX-J" H 2250 2825 50  0001 C CNN
+F 2 "Capacitor_Tantalum_SMD:CP_EIA-2012-15_AVX-P_Pad1.30x1.05mm_HandSolder" H 2250 2825 50  0001 C CNN
 F 3 "~" H 2250 2825 50  0001 C CNN
 	1    2250 2825
@@
 F 0 "C2" H 1140 2821 50  0000 L CNN
 F 1 "100n" H 1140 2730 50  0000 L CNN
-F 2 "Capacitor_Tantalum_SMD:CP_EIA-1608-08_AVX-J" H 1025 2775 50  0001 C CNN
+F 2 "Capacitor_Tantalum_SMD:CP_EIA-2012-15_AVX-P_Pad1.30x1.05mm_HandSolder" H 1025 2775 50  0001 C CNN
 F 3 "~" H 1025 2775 50  0001 C CNN
 	1    1025 2775
